File: 2 PCB/CircuitBoard/CircuitBoardV2.kicad_pcb (KiCad board)
At the start: 2 copper layers, 57.4 x 132.3 mm, 53 parts, among them J1 Conn_01x04_Male, J10 Conn_01x04_Male, J11 Conn_01x04_Male, J12 Conn_01x04_Male, J13 Conn_01x04_Male, J14 Conn_01x04_Male, J15 Conn_01x04_Male, J16 Conn_01x04_Male, J17 Conn_01x04_Male, J18 Conn_01x04_Male, J19 Conn_01x04_Male, J2 Conn_01x04_Male, J20 Conn_01x04_Male, J21 Conn_01x24_Female, J22 Conn_01x24_Female, J23 Conn_01x04_Male, J24 Conn_01x04_Male, J25 Conn_01x04_Male, J26 Conn_01x04_Male, J27 Conn_01x04_Male, J28 Conn_01x04_Male, J29 Conn_01x04_Male, J3 Conn_01x04_Male, J30 Conn_01x04_Male, J31 Conn_01x04_Male, J32 Conn_01x04_Male, J33 Conn_01x04_Male, J34 Conn_01x04_Male, J35 Conn_01x04_Male, J36 Conn_01x04_Male, J37 Conn_01x04_Male, J38 Conn_01x04_Male, J39 Conn_01x04_Male, J4 Conn_01x04_Male, J40 Conn_01x04_Male, J41 Conn_01x04_Male, J42 Conn_01x04_Male, J5 Conn_01x04_Male, J6 Conn_01x04_Male, J7 Conn_01x04_Male, J8 Conn_01x04_Male, J9 Conn_01x04_Male, U1 TXS0108EPWR, U2 TXS0108EPWR, U3 TXS0108EPWR, U4 TXS0108EPWR, U5 TXS0108EPWR

Commit message: New Patterns and New Features and Deployment
Some changes as it was fully deployed and I was able to test everything. I was concerned about the temperature of the teensy so I added another serial command to check the internal temperature of the teensy. I was also testing out a ton of patterns major trial and error.
Other:
- net class Default removed
